Commit message: Add more files for alunching with ros2_control and rviz

File: karp_description/ros2_control/karp_system.ros2_control.xacro (robot description, xacro)
@@ -1,12 +1,16 @@
 <?xml version="1.0"?>
 <robot xmlns:xacro="http://www.ros.org/wiki/xacro">
-  <xacro:macro name="karp_ros2_control" params="name prefix">
+  <xacro:macro name="karp_system" params="name prefix use_fake_hardware:=^|false fake_sensor_commands:=^|false">
     <ros2_control name="${name}" type="system">
       <hardware>
-        <plugin>odrive_hardware_interface/ODriveHardwareInterface</plugin>
+        <xacro:if value="${use_fake_hardware}">
+          <plugin>fake_components/GenericSystem</plugin>
+          <param name="fake_sensor_commands">${fake_sensor_commands}</param>
+          <param name="state_following_offset">0.0</param>
+        </xacro:if>
+        <xacro:unless value="${use_fake_hardware}">
+          <plugin>odrive_hardware_interface/ODriveHardwareInterface</plugin>
+        </xacro:unless>
       </hardware>
-      <sensor name="odrv0">
-        <param name="serial_number">000000000000</param>
-      </sensor>
       <joint name="${prefix}left_wheel_joint">
         <command_interface name="velocity"/>
