Commit message: Update parameters

File: karp_description/urdf/karp_description.urdf.xacro (robot description, xacro)
@@ -4,13 +4,13 @@
   <!-- Constants for robot dimensions -->
   <xacro:property name="PI" value="3.1415926535897931"/>
-  <xacro:property name="base_mass" value="0.3" /> <!-- arbitrary value for base mass -->
+  <xacro:property name="base_mass" value="5" /> <!-- arbitrary value for base mass -->
   <xacro:property name="base_width" value="0.36" />
   <xacro:property name="base_length" value="0.51" />
-  <xacro:property name="base_height" value="0.2" />
-  <xacro:property name="wheel_mass" value="0.3" /> <!-- arbitrary value for wheel mass -->
-  <xacro:property name="wheel_len" value="0.020" />
-  <xacro:property name="wheel_radius" value="0.015" />
-  <xacro:property name="caster_wheel_mass" value="0.1" /> <!-- arbitrary value for caster wheel mass -->
-  <xacro:property name="caster_wheel_radius" value="0.015" />
+  <xacro:property name="base_height" value="0.20" />
+  <xacro:property name="wheel_mass" value="2.2" />
+  <xacro:property name="wheel_len" value="0.045" />
+  <xacro:property name="wheel_radius" value="0.085" />
+  <xacro:property name="caster_wheel_mass" value="2.1" />
+  <xacro:property name="caster_wheel_radius" value="0.08" />
   <xacro:property name="z_offset" value="-${base_height/2}" /> <!-- Space btw top of beam and the each joint -->
   <!-- Base Link -->

Commit message: Update robot description and rviz config

File: karp_description/urdf/karp_description.urdf.xacro (robot description, xacro)
@@ -17,5 +17,5 @@
   <link name="${prefix}base_link">
     <collision>
-      <origin xyz="0 0 0" rpy="0 0 0"/>
+      <origin xyz="0 0 ${base_height/2}" rpy="0 0 ${PI/2}"/>
       <geometry>
         <box size="${base_width} ${base_length} ${base_height}"/>
@@ -23,5 +23,5 @@
     </collision>
     <visual>
-      <origin xyz="0 0 0" rpy="${PI/2}  0 0"/>
+      <origin xyz="0 0 0" rpy="${PI/2}  0 ${PI/2}"/>
       <geometry>
         <mesh filename="package://karp_description/meshes/KARP_body.dae" />
@@ -41,6 +41,6 @@
     <parent link="${prefix}base_link"/>
     <child link="${prefix}left_wheel"/>
-    <origin xyz="0.119 -0.165 -0.11975" rpy="0 0 0"/>
-    <axis xyz="1 0 0"/>
+    <origin xyz="0.165 -0.119 -0.11975" rpy="0 0 0"/>
+    <axis xyz="0 1 0"/>
     <dynamics damping="0.2"/>
   </joint>
@@ -48,5 +48,5 @@
   <link name="${prefix}left_wheel">
     <collision>
-      <origin xyz="0 0 0" rpy="0 0 0"/>
+      <origin xyz="0 ${wheel_len/2} 0" rpy="${PI/2} 0 0"/>
       <geometry>
         <cylinder length="${wheel_len}" radius="${wheel_radius}"/>
@@ -54,5 +54,5 @@
     </collision>
     <visual>
-      <origin xyz="0 0 0" rpy="0  0 0"/>
+      <origin xyz="0 0 0" rpy="0 0 -${PI/2}"/>
       <geometry>
         <mesh filename="package://karp_description/meshes/KARP_left_wheel.dae" />
@@ -72,6 +72,6 @@
     <parent link="${prefix}base_link"/>
     <child link="${prefix}right_wheel"/>
-    <origin xyz="-0.119 -0.165 -0.11975" rpy="0 0 0"/>
-    <axis xyz="1 0 0"/>
+    <origin xyz="0.165 0.119 -0.11975" rpy="0 0 0"/>
+    <axis xyz="0 1 0"/>
     <dynamics damping="0.2"/>
   </joint>
@@ -79,5 +79,5 @@
   <link name="${prefix}right_wheel">
     <collision>
-      <origin xyz="0 0 0" rpy="0 0 0"/>
+      <origin xyz="0 -${wheel_len/2} 0" rpy="${PI/2} 0 0"/>
       <geometry>
         <cylinder length="${wheel_len}" radius="${wheel_radius}"/>
@@ -85,9 +85,8 @@
     </collision>
     <visual>
-      <origin xyz="0 0 0" rpy="0 0 0"/>
+      <origin xyz="0 0 0" rpy="0 0 ${PI/2}"/>
       <geometry>
-        <mesh filename="package://karp_description/meshes/KARP_right_wheel.dae" />
+        <mesh filename="package://karp_description/meshes/KARP_left_wheel.dae" />
       </geometry>
-      <material name="black"/>
     </visual>
     <inertial>
@@ -104,10 +103,10 @@
     <parent link="${prefix}base_link"/>
     <child link="${prefix}caster_left_wheel"/>
-    <origin xyz="0.165 0.216 -0.028" rpy="0 0 0"/>
+    <origin xyz="-0.216 0.165 -0.028" rpy="0 0 0"/>
   </joint>
   <!-- caster left wheel Link -->
   <link name="${prefix}caster_left_wheel">
     <collision>
-      <origin xyz="0 0 0" rpy="0 0 0"/>
+      <origin xyz="0.052 0 -0.1" rpy="0 0 0"/>
       <geometry>
         <sphere radius="${caster_wheel_radius}"/>
@@ -115,9 +114,8 @@
     </collision>
     <visual>
-      <origin xyz="0 0 0" rpy="${PI/2}  0 0"/>
+      <origin xyz="0 0 0" rpy="${PI/2}  0 ${PI/2}"/>
       <geometry>
         <mesh filename="package://karp_description/meshes/KARP_caster_wheel.dae" />
       </geometry>
-      <material name="white"/>
     </visual>
     <inertial>
@@ -134,10 +132,10 @@
     <parent link="${prefix}base_link"/>
     <child link="${prefix}caster_right_wheel"/>
-    <origin xyz="-0.165 0.216 -0.028" rpy="0 0 0"/>
+    <origin xyz="-0.216 -0.165  -0.028" rpy="0 0 0"/>
   </joint>
   <!-- caster right wheel Link -->
   <link name="${prefix}caster_right_wheel">
     <collision>
-      <origin xyz="0 0 0" rpy="0 0 0"/>
+      <origin xyz="0.052 0 -0.1" rpy="0 0 0"/>
       <geometry>
         <sphere radius="${caster_wheel_radius}"/>
@@ -145,9 +143,8 @@
     </collision>
     <visual>
-      <origin xyz="0 0 0" rpy="${PI/2}  0 0"/>
+      <origin xyz="0 0 0" rpy="${PI/2}  0 ${PI/2}"/>
       <geometry>
         <mesh filename="package://karp_description/meshes/KARP_caster_wheel.dae" />
       </geometry>
-      <material name="white"/>
     </visual>
     <inertial>
@@ -164,10 +161,10 @@
     <parent link="${prefix}base_link"/>
     <child link="${prefix}base_laser"/>
-    <origin xyz="0 -0.151 0.208" rpy="0 0 0"/>
+    <origin xyz="0.151 0 0.208" rpy="0 0 0"/>
   </joint>
   <!-- lidar link-->
   <link name="${prefix}base_laser">
     <visual>
-      <origin xyz="0 0 0" rpy="${PI/2} 0 0"/>
+      <origin xyz="0 0 0" rpy="${PI/2} 0 ${PI/2}"/>
       <geometry>
         <mesh filename="package://karp_description/meshes/velodyne.dae" />

Commit message: Unify wheel dae and remove one wheel dae file

File: karp_description/urdf/karp_description.urdf.xacro (robot description, xacro)
@@ -56,5 +56,5 @@
       <origin xyz="0 0 0" rpy="0 0 -${PI/2}"/>
       <geometry>
-        <mesh filename="package://karp_description/meshes/KARP_left_wheel.dae" />
+        <mesh filename="package://karp_description/meshes/KARP_wheel.dae" />
       </geometry>
     </visual>
@@ -87,5 +87,5 @@
       <origin xyz="0 0 0" rpy="0 0 ${PI/2}"/>
       <geometry>
-        <mesh filename="package://karp_description/meshes/KARP_left_wheel.dae" />
+        <mesh filename="package://karp_description/meshes/KARP_wheel.dae" />
       </geometry>
     </visual>
