Commit message: Update Velodyne lidar in KARP URDF

File: karp_description/urdf/karp.urdf.xacro (robot description, xacro)
@@ -6,5 +6,10 @@
   <!-- Import karp ros2_control description -->
   <xacro:include filename="$(find karp_description)/ros2_control/karp.ros2_control.xacro" />
+  <!-- Import velodyne VLP16 description -->
+  <xacro:include filename="$(find karp_description)/urdf/VLP-16.urdf.xacro"/>
   <xacro:karp prefix="$(arg prefix)" />
   <xacro:karp_ros2_control name="karp" prefix="$(arg prefix)" />
+  <xacro:VLP-16 parent="$(arg prefix)base_link" name="velodyne">
+    <origin xyz="0.151 0 0.208" rpy="0 0 0"/>
+  </xacro:VLP-16>
 </robot>

File: karp_description/urdf/karp_description.urdf.xacro (robot description, xacro)
@@ -157,19 +157,4 @@
     </inertial>
   </link>
-  <!-- lidar joint-->
-  <joint name="${prefix}lidar_joint" type="fixed">
-    <parent link="${prefix}base_link"/>
-    <child link="${prefix}base_laser"/>
-    <origin xyz="0.151 0 0.208" rpy="0 0 0"/>
-  </joint>
-  <!-- lidar link-->
-  <link name="${prefix}base_laser">
-    <visual>
-      <origin xyz="0 0 0" rpy="${PI/2} 0 ${PI/2}"/>
-      <geometry>
-        <mesh filename="package://karp_description/meshes/velodyne.dae" />
-      </geometry>
-    </visual>
-  </link>
   </xacro:macro>
 </robot>

File: karp_description/urdf/karp_system.urdf.xacro (robot description, xacro)
@@ -8,13 +8,15 @@
   <xacro:arg name="prefix" default="" />
   <xacro:include filename="$(find karp_description)/urdf/karp_description.urdf.xacro" />
-  <!-- Import all Gazebo-customization elements, including Gazebo colors -->
-  <!-- <xacro:include filename="$(find karp_description)/gazebo/karp.gazebo.xacro" /> -->
   <!-- Import karp ros2_control description -->
   <xacro:include filename="$(find karp_description)/ros2_control/karp_system.ros2_control.xacro" />
+  <!-- Import velodyne VLP16 description -->
+  <xacro:include filename="$(find karp_description)/urdf/VLP-16.urdf.xacro"/>
   <xacro:karp prefix="$(arg prefix)" />
-  <!-- <xacro:karp_gazebo prefix="$(arg prefix)" /> -->
   <xacro:karp_system
     name="KARPSystem" prefix="$(arg prefix)"
     use_fake_hardware="$(arg use_fake_hardware)"
     fake_sensor_commands="$(arg fake_sensor_commands)"/>
+  <xacro:VLP-16 parent="$(arg prefix)base_link" name="velodyne">
+    <origin xyz="0.151 0 0.208" rpy="0 0 0"/>
+  </xacro:VLP-16>
 </robot>
